File: nRF52832_MCU.brd (EAGLE design)
At the start: 35.2 x 23.3 mm, 31 parts, among them J100 DEBUG_CONNECTOR, P1 WIREPADSMD1,27-254, P2 WIREPADSMD1,27-254, P3 WIREPADSMD1,27-254, P4 WIREPADSMD1,27-254, U1 NRF52832, X1 32MHz, X2 32.768kHz

Commit message: Add coplanar computation
Parts:
- moved C5 0.11 mm to (23.7, 15.5)
- moved C8 0.07 mm to (24.5, 13.5)
Connections:
- net GND renamed N$10
